File: USB-C PD Trigger (Programmable Bench Supply).kicad_pcb (KiCad board)
At the start: 2 copper layers, 30 x 35 mm, 17 parts, among them J2 Conn_01x01_Socket, J3 Conn_01x01_Socket, J4 Conn_02x04_Counter_Clockwise, J5 USB_C_Receptacle, U1 CH224K

Commit message: schematics Organized
Connections:
- net /CFG1 renamed /CFG_1
- net Net-(J5-CC1) renamed /CC1
- net Net-(J5-CC2) renamed /CC2
- J4 pad 4: unconnected-(J4-Pin_4-Pad4) -> /VDD
Routing:
- net /VDD: track 13.5 -> 31.6 mm, vias 0 -> 1

Commit message: 5v label added to jumper & updated readme.md
Parts:
- moved C1 21.3 mm to (47.3, 53.4)
- moved J5 21.3 mm to (52.0, 59.5)
- moved C2 21.3 mm to (57.1, 53.4)
- moved C3 21.3 mm to (51.6, 44.1)
- moved D1 21.3 mm to (44.0, 53.2)
- moved J2 21.3 mm to (44.4, 44.1)
- moved J3 21.3 mm to (58.9, 44.1)
- moved J4 21.3 mm to (65.1, 63.7)
- moved R1 21.3 mm to (44.5, 59.4)
- moved R2 21.3 mm to (44.5, 61.0)
- moved R3 21.3 mm to (58.0, 55.9)
- moved R4 21.3 mm to (58.0, 57.5)
- moved R5 21.3 mm to (45.6, 53.4)
- moved R8 21.3 mm to (63.1, 60.3)
- moved R9 21.3 mm to (61.1, 60.3)
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Other:
- board text added: "5v"
